File: pcb/controller_ic.sch (KiCad schematic (older format))
At the start: 0 parts

Commit message: SCH: missing signal logic and level shifting
Parts:
- added C? (x2): 27pF, symbol Device:C_Small
- added C? (x10): 100nF, symbol Device:C_Small
- added C? (x2): 4.7uF, symbol Device:C_Small
- added FB? (x2): nH, symbol Device:Ferrite_Bead_Small
- added R?: 12K, symbol Device:R_Small
- added R?: 1k, symbol Device:R_Small
- added R?: 2k, symbol Device:R_Small
- added R? (x3): 10k, symbol Device:R_Small
- added U?: FT4232H, symbol Interface_USB:FT4232H
- added U?: 93LCxxBxxOT, Package_TO_SOT_SMD:SOT-23-6, symbol Memory_EEPROM:93LCxxBxxOT
- added Y?: 12MHz, symbol Device:Crystal
Connections:
- new net: R?.2, U?.14 (~RESET)
- new net: C?.1, U?.2 (OSCI), Y?.1
- new net: C?.1, U?.3 (OSCO), Y?.2
- new net: C?.1, C?.1, FB?.2, U?.4 (VPHY)
- new net: R?.1, U?.6 (REF)
- new net: R?.2, U?.3 (DI), U?.61 (EEDATA)
- new net: R?.2, U?.4 (CLK), U?.62 (EECLK)
- new net: C?.1, C?.1, FB?.2, U?.9 (VPLL)
- new net: R?.1, R?.2, U?.1 (DO)
- new net +1V8: C?.1, C?.1, C?.1, U?.12 (VCORE), U?.37 (VCORE), U?.64 (VCORE)
- new net +3V3: C?.1, C?.1, C?.1, C?.1, C?.1, FB?.1, FB?.1, R?.1, R?.1, R?.1, R?.1, U?.20 (VCCIO), U?.31 (VCCIO), U?.42 (VCCIO), U?.56 (VCCIO), U?.6 (VCC)
- new net ADBUS0: U?.16 (ADBUS0)
- new net ADBUS1: U?.17 (ADBUS1)
- new net ADBUS2: U?.18 (ADBUS2)
- new net ADBUS3: U?.19 (ADBUS3)
- new net ADBUS4: U?.21 (ADBUS4)
- new net ADBUS5: U?.22 (ADBUS5)
- new net ADBUS6: U?.23 (ADBUS6)
- new net ADBUS7: U?.24 (ADBUS7)
- new net BDBUS0: U?.26 (BDBUS0)
- new net BDBUS1: U?.27 (BDBUS1)
- new net BDBUS2: U?.28 (BDBUS2)
- new net BDBUS3: U?.29 (BDBUS3)
- new net BDBUS4: U?.30 (BDBUS4)
- new net BDBUS5: U?.32 (BDBUS5)
- new net BDBUS6: U?.33 (BDBUS6)
- new net BDBUS7: U?.34 (BDBUS7)
- new net CDBUS0: U?.38 (CDBUS0)
- new net CDBUS1: U?.39 (CDBUS1)
- new net CDBUS2: U?.40 (CDBUS2)
- new net CDBUS3: U?.41 (CDBUS3)
- new net CDBUS4: U?.43 (CDBUS4)
- new net CDBUS5: U?.44 (CDBUS5)
- new net CDBUS6: U?.45 (CDBUS6)
- new net CDBUS7: U?.46 (CDBUS7)
- new net DDBUS0: U?.48 (DDBUS0)
- new net DDBUS1: U?.52 (DDBUS1)
- new net DDBUS2: U?.53 (DDBUS2)
- new net DDBUS3: U?.54 (DDBUS3)
- new net DDBUS4: U?.55 (DDBUS4)
- new net DDBUS5: U?.57 (DDBUS5)
- new net DDBUS6: U?.58 (DDBUS6)
- new net DDBUS7: U?.59 (DDBUS7)
- new net DM: U?.7 (DM)
- new net DP: U?.8 (DP)
- new net EECS: R?.2, U?.5 (CS), U?.63 (EECS)
- new net GND: C?.2, C?.2, C?.2, C?.2, C?.2, C?.2, C?.2, C?.2, C?.2, C?.2, C?.2, C?.2, C?.2, C?.2, R?.2, U?.1 (GND), U?.10 (AGND), U?.11 (GND), U?.13 (TEST), U?.15 (GND), U?.2 (GND), U?.25 (GND), U?.35 (GND), U?.47 (GND), U?.5 (GND), U?.51 (GND)
- no-connect marks 0 -> 2
Other:
- note added: "MPSSE"
