File: pcb/controller_ic.sch (KiCad schematic (older format))
At the start: 25 parts

Commit message: SCH: minor changes
Parts:
- added C?: 4.7uF, symbol Device:C_Small
- added C?: 100nF, symbol Device:C_Small
Connections:
- net +1V8: now also U?.49 (VREGOUT), C?.1
- net +3V3: now also U?.50 (VREGIN), C?.1
- net GND: now also C?.2, C?.2
- no-connect marks 2 -> 0
Changed lines of the file:
@@
 	1    0    0    -1
 $EndComp
-NoConn ~ 3300 2800
-NoConn ~ 3300 2600
 $Comp
 L power:+3V3 #PWR?
@@
 Text Notes 5150 4200 1    50   ~ 0
 MPSSE
-Wire Bus Line
-	6150 5150 6150 5900
-Wire Bus Line
-	6150 4250 6150 5000
-Wire Bus Line
-	6150 3350 6150 4100
-Wire Bus Line
-	6150 2450 6150 3200
 $Bitmap
 Pos 9250 4050
@@
 EndData
 $EndBitmap
+Wire Wire Line
+	3300 2600 2450 2600
+Wire Wire Line
+	2450 2600 2450 2400
+$Comp
+L power:+3V3 #PWR?
+U 1 1 5E70B267
+P 2450 2400
+F 0 "#PWR?" H 2450 2250 50  0001 C CNN
+F 1 "+3V3" H 2465 2573 50  0000 C CNN
+F 2 "" H 2450 2400 50  0001 C CNN
+F 3 "" H 2450 2400 50  0001 C CNN
+	1    2450 2400
+	1    0    0    -1
+$EndComp
+$Comp
+L Device:C_Small C?
+U 1 1 5E70B729
+P 2450 2900
+F 0 "C?" H 2200 2950 50  0000 L CNN
+F 1 "4.7uF" H 2150 2850 50  0000 L CNN
+F 2 "" H 2450 2900 50  0001 C CNN
+F 3 "~" H 2450 2900 50  0001 C CNN
+	1    2450 2900
+	1    0    0    -1
+$EndComp
+Wire Wire Line
+	2450 2800 2450 2600
+Connection ~ 2450 2600
+Wire Wire Line
+	2450 3000 2450 3100
+$Comp
+L power:GND #PWR?
+U 1 1 5E719122
+P 2450 3100
+F 0 "#PWR?" H 2450 2850 50  0001 C CNN
+F 1 "GND" H 2455 2927 50  0000 C CNN
+F 2 "" H 2450 3100 50  0001 C CNN
+F 3 "" H 2450 3100 50  0001 C CNN
+	1    2450 3100
+	1    0    0    -1
+$EndComp
+Wire Wire Line
+	3300 2800 3250 2800
+Wire Wire Line
+	3250 2800 3250 2900
+Wire Wire Line
+	3250 2900 3100 2900
+Wire Wire Line
+	3100 2900 3100 2850
+$Comp
+L power:+1V8 #PWR?
+U 1 1 5E71FE15
+P 3100 2850
+F 0 "#PWR?" H 3100 2700 50  0001 C CNN
+F 1 "+1V8" H 3115 3023 50  0000 C CNN
+F 2 "" H 3100 2850 50  0001 C CNN
+F 3 "" H 3100 2850 50  0001 C CNN
+	1    3100 2850
+	1    0    0    -1
+$EndComp
+Wire Wire Line
+	3250 3200 3250 3250
+$Comp
+L Device:C_Small C?
+U 1 1 5E72D936
+P 3250 3100
+F 0 "C?" H 3000 3150 50  0000 L CNN
+F 1 "100nF" H 2900 3050 50  0000 L CNN
+F 2 "" H 3250 3100 50  0001 C CNN
+F 3 "~" H 3250 3100 50  0001 C CNN
+	1    3250 3100
+	1    0    0    -1
+$EndComp
+$Comp
+L power:GND #PWR?
+U 1 1 5E72D93C
+P 3250 3250
+F 0 "#PWR?" H 3250 3000 50  0001 C CNN
+F 1 "GND" H 3255 3077 50  0000 C CNN
+F 2 "" H 3250 3250 50  0001 C CNN
+F 3 "" H 3250 3250 50  0001 C CNN
+	1    3250 3250
+	1    0    0    -1
+$EndComp
+Wire Wire Line
+	3250 3000 3250 2900
+Wire Bus Line
+	6150 5150 6150 5900
+Wire Bus Line
+	6150 4250 6150 5000
+Wire Bus Line
+	6150 3350 6150 4100
+Wire Bus Line
+	6150 2450 6150 3200
+Connection ~ 3250 2900
 $EndSCHEMATC

Commit message: SCH: slight changes
Parts:
- removed Y?: 12MHz, symbol Device:Crystal
- added Y201: 12MHz, Crystal:Crystal_SMD_3225-4Pin_3.2x2.5mm_HandSoldering, symbol Device:Crystal_GND23
- C201, C202, C203, C204, C205, C206, C207, C208, C209, C210, C211, C212, C213, C214, C215, C216: renamed from C?; footprint (none) -> Capacitor_SMD:C_0603_1608Metric_Pad1.05x0.95mm_HandSolder
- FB201, FB202: renamed from FB?; value nH -> 600R/0.5A; footprint (none) -> Inductor_SMD:L_0603_1608Metric_Pad1.05x0.95mm_HandSolder
- R201, R202, R203, R204, R205, R206: renamed from R?; footprint (none) -> Resistor_SMD:R_0603_1608Metric_Pad1.05x0.95mm_HandSolder
- U202: renamed from U?; footprint (none) -> Package_QFP:LQFP-64_10x10mm_P0.5mm
- gave numbers to parts that had none: 1
Connections:
- net GND: now also Y201.2, Y201.3
- net at C202.1, U202.2 (OSCI): now also Y201.1
- net at C204.1, U202.3 (OSCO): now also Y201.4
- no-connect marks 0 -> 2
Other:
- moved on the sheet: C202, C204
