File: pcb/power.sch (KiCad schematic (older format))
At the start: 0 parts

Commit message: SCH: missing signal logic and level shifting
Parts:
- added C? (x2): 1uF, symbol Device:C_Small
- added C? (x4): 4.7uF, symbol Device:C_Small
- added C?: 470pF, symbol Device:C_Small
- added C?: C_Small, symbol Device:C_Small
- added L? (x2): 1uH, symbol Device:L_Small
- added R? (x2): 100kΩ, symbol Device:R_Small
- added R?: 71.5kΩ, symbol Device:R_Small
- added R?: 309kΩ, symbol Device:R_Small
- added R?: 158kΩ, symbol Device:R_Small
- added R?: 301kΩ, symbol Device:R_Small
- added U?: MIC23159, symbol rs_Regulator_switching:MIC23159
Connections:
- new net: R?.1, R?.2, U?.11 (FB2)
- new net: C?.1, U?.13 (SS2)
- new net: C?.1, U?.14 (SS1)
- new net: R?.2, R?.2, U?.16 (FB1)
- new net: R?.1, U?.18 (EN1)
- new net: L?.2, U?.3 (SW1)
- new net: L?.1, U?.4 (SW2)
- new net: R?.2, U?.9 (EN2)
- new net +1V8: C?.1, L?.2, R?.1, U?.10 (SNS2)
- new net +3V3: C?.1, L?.1, R?.1, U?.17 (SNS1)
- new net GND: C?.2, C?.2, C?.2, C?.2, C?.2, C?.2, C?.2, C?.2, R?.1, R?.2, U?.19 (AGND1), U?.2 (PGND1), U?.5 (PGND2), U?.~ (PAD)
- new net VBUS: C?.1, C?.1, C?.1, C?.1, R?.1, R?.2, U?.1 (VIN1), U?.20 (AVIN1), U?.6 (VIN2), U?.7 (AVIN2)
Other:
- note added: "Switched Power Regulator"
