File: pcb/power.sch (KiCad schematic (older format))
At the start: 17 parts

Commit message: SCH: minor changes
Parts:
- removed C?: 1uF, symbol Device:C_Small
- removed C? (x2): 4.7uF, symbol Device:C_Small
- removed C?: C_Small, symbol Device:C_Small
- removed L? (x2): 1uH, symbol Device:L_Small
- removed R?: 100kΩ, symbol Device:R_Small
- removed R?: 158kΩ, symbol Device:R_Small
- removed R?: 301kΩ, symbol Device:R_Small
- removed U?: MIC23159, symbol rs_Regulator_switching:MIC23159
- added L?: 1uH, symbol Device:L
- added U?: MIC23155, symbol rs_Regulator_switching:MIC23155
Connections:
- net +3V3: now also L?.1, U?.3 (SNS)
- net GND: now also U?.10 (PGND), U?.11 (ePAD), U?.7 (AGND)
- net VBUS: now also U?.8 (VIN), U?.9 (VIN)
- net at C?.1: now also U?.6 (SS)
- net at R?.2, R?.2: now also U?.16 (FB)
- net at R?.1: now also U?.2 (EN)
- new net: L?.2, U?.1 (SW)
- no-connect marks 0 -> 1
Other:
- moved on the sheet: C?, R?

Commit message: SCH: slight changes
Parts:
- added C505: 100nF, Capacitor_SMD:C_0603_1608Metric_Pad1.05x0.95mm_HandSolder, symbol Device:C_Small
- C501, C503, C504: renamed from C?; footprint (none) -> Capacitor_SMD:C_0603_1608Metric_Pad1.05x0.95mm_HandSolder
- C502: renamed from C?; value 1uF -> 100nF; footprint (none) -> Capacitor_SMD:C_0603_1608Metric_Pad1.05x0.95mm_HandSolder
- L501: renamed from L?; footprint (none) -> Inductor_SMD:L_0805_2012Metric_Pad1.15x1.40mm_HandSolder
- R501, R502, R503: renamed from R?; footprint (none) -> Resistor_SMD:R_0603_1608Metric_Pad1.05x0.95mm_HandSolder
- U501: renamed from U?; footprint (none) -> mic23155:MLF-20-1EP_3x4mm_P0.5mm_EP2.6x1.6mm_thermal_vias
Connections:
- net +3V3: now also C505.1
- net GND: now also C505.2
Other:
- moved on the sheet: C504
Changed lines of the file:
@@
 	5600 4100 5600 4200
 $Comp
-L power:GND #PWR?
+L power:GND #PWR0505
 U 1 1 5E8A218D
 P 5600 4200
-F 0 "#PWR?" H 5600 3950 50  0001 C CNN
+F 0 "#PWR0505" H 5600 3950 50  0001 C CNN
 F 1 "GND" H 5605 4027 50  0000 C CNN
 F 2 "" H 5600 4200 50  0001 C CNN
@@
 $EndComp
 $Comp
-L Device:C_Small C?
+L Device:C_Small C504
 U 1 1 5E8C0ADA
-P 7300 3600
-F 0 "C?" H 7050 3650 50  0000 L CNN
-F 1 "4.7uF" H 6950 3550 50  0000 L CNN
-F 2 "" H 7300 3600 50  0001 C CNN
-F 3 "~" H 7300 3600 50  0001 C CNN
-	1    7300 3600
-	-1   0    0    -1
-$EndComp
-$Comp
-L Device:C_Small C?
+P 7700 3600
+F 0 "C504" H 7450 3650 50  0000 L CNN
+F 1 "4.7uF" H 7350 3550 50  0000 L CNN
+F 2 "Capacitor_SMD:C_0603_1608Metric_Pad1.05x0.95mm_HandSolder" H 7700 3600 50  0001 C CNN
+F 3 "~" H 7700 3600 50  0001 C CNN
+	1    7700 3600
+	-1   0    0    -1
+$EndComp
+$Comp
+L Device:C_Small C503
 U 1 1 5E8C1191
 P 6250 4100
-F 0 "C?" H 6342 4146 50  0000 L CNN
+F 0 "C503" H 6342 4146 50  0000 L CNN
 F 1 "470pF" H 6342 4055 50  0000 L CNN
-F 2 "" H 6250 4100 50  0001 C CNN
+F 2 "Capacitor_SMD:C_0603_1608Metric_Pad1.05x0.95mm_HandSolder" H 6250 4100 50  0001 C CNN
 F 3 "~" H 6250 4100 50  0001 C CNN
 	1    6250 4100
@@
 $EndComp
 $Comp
-L Device:R_Small R?
+L Device:R_Small R501
 U 1 1 5E8C1A3D
 P 5000 3800
-F 0 "R?" V 5100 3800 50  0000 C CNN
+F 0 "R501" V 5100 3800 50  0000 C CNN
 F 1 "100kΩ" V 4900 3800 50  0000 C CNN
-F 2 "" H 5000 3800 50  0001 C CNN
+F 2 "Resistor_SMD:R_0603_1608Metric_Pad1.05x0.95mm_HandSolder" H 5000 3800 50  0001 C CNN
 F 3 "~" H 5000 3800 50  0001 C CNN
 	1    5000 3800
@@
 $EndComp
 $Comp
-L Device:R_Small R?
+L Device:R_Small R502
 U 1 1 5E8C239B
 P 6600 3800
-F 0 "R?" H 6850 3750 50  0000 R CNN
+F 0 "R502" H 6850 3750 50  0000 R CNN
 F 1 "71.5kΩ" H 7000 3850 50  0000 R CNN
-F 2 "" H 6600 3800 50  0001 C CNN
+F 2 "Resistor_SMD:R_0603_1608Metric_Pad1.05x0.95mm_HandSolder" H 6600 3800 50  0001 C CNN
 F 3 "~" H 6600 3800 50  0001 C CNN
 	1    6600 3800
@@
 $EndComp
 $Comp
-L Device:R_Small R?
+L Device:R_Small R503
 U 1 1 5E8C27EB
 P 6800 3600
-F 0 "R?" V 6900 3750 50  0000 C CNN
+F 0 "R503" V 6900 3750 50  0000 C CNN
 F 1 "309kΩ" V 6900 3450 50  0000 C CNN
-F 2 "" H 6800 3600 50  0001 C CNN
+F 2 "Resistor_SMD:R_0603_1608Metric_Pad1.05x0.95mm_HandSolder" H 6800 3600 50  0001 C CNN
 F 3 "~" H 6800 3600 50  0001 C CNN
 	1    6800 3600
@@
 $EndComp
 $Comp
-L power:VBUS #PWR?
+L power:VBUS #PWR0504
 U 1 1 5E8D4A49
 P 4800 3700
-F 0 "#PWR?" H 4800 3550 50  0001 C CNN
+F 0 "#PWR0504" H 4800 3550 50  0001 C CNN
 F 1 "VBUS" H 4700 3850 50  0000 L CNN
 F 2 "" H 4800 3700 50  0001 C CNN
@@
 	7100 3600 7100 3400
 Wire Wire Line
-	7100 3400 7300 3400
-Wire Wire Line
-	7300 3400 7300 3300
+	7100 3400 7500 3400
+Wire Wire Line
+	7700 3400 7700 3300
 Connection ~ 7100 3400
 Wire Wire Line
 	7100 3200 7100 3400
 Wire Wire Line
-	7300 3400 7300 3500
-Connection ~ 7300 3400
-$Comp
-L power:GND #PWR?
+	7700 3400 7700 3500
+Connection ~ 7700 3400
+$Comp
+L power:GND #PWR0509
 U 1 1 5E8DB0E1
-P 7300 3800
-F 0 "#PWR?" H 7300 3550 50  0001 C CNN
-F 1 "GND" H 7305 3627 50  0000 C CNN
-F 2 "" H 7300 3800 50  0001 C CNN
-F 3 "" H 7300 3800 50  0001 C CNN
-	1    7300 3800
-	-1   0    0    -1
-$EndComp
-$Comp
-L power:GND #PWR?
+P 7700 3800
+F 0 "#PWR0509" H 7700 3550 50  0001 C CNN
+F 1 "GND" H 7705 3627 50  0000 C CNN
+F 2 "" H 7700 3800 50  0001 C CNN
+F 3 "" H 7700 3800 50  0001 C CNN
+	1    7700 3800
+	-1   0    0    -1
+$EndComp
+$Comp
+L power:GND #PWR0507
 U 1 1 5E8DB4DB
 P 6600 4000
-F 0 "#PWR?" H 6600 3750 50  0001 C CNN
+F 0 "#PWR0507" H 6600 3750 50  0001 C CNN
 F 1 "GND" H 6605 3827 50  0000 C CNN
 F 2 "" H 6600 4000 50  0001 C CNN
@@
 	6600 4000 6600 3900
 Wire Wire Line
-	7300 3800 7300 3700
-$Comp
-L power:+3V3 #PWR?
+	7700 3800 7700 3700
+$Comp
+L power:+3V3 #PWR0508
 U 1 1 5E8DC866
-P 7300 3300
-F 0 "#PWR?" H 7300 3150 50  0001 C CNN
-F 1 "+3V3" H 7315 3473 50  0000 C CNN
-F 2 "" H 7300 3300 50  0001 C CNN
-F 3 "" H 7300 3300 50  0001 C CNN
-	1    7300 3300
+P 7700 3300
+F 0 "#PWR0508" H 7700 3150 50  0001 C CNN
+F 1 "+3V3" H 7715 3473 50  0000 C CNN
+F 2 "" H 7700 3300 50  0001 C CNN
+F 3 "" H 7700 3300 50  0001 C CNN
+	1    7700 3300
 	-1   0    0    -1
 $EndComp
@@
 	6250 3800 6050 3800
 $Comp
-L power:GND #PWR?
+L power:GND #PWR0506
 U 1 1 5E8DE7FB
 P 6250 4300
-F 0 "#PWR?" H 6250 4050 50  0001 C CNN
+F 0 "#PWR0506" H 6250 4050 50  0001 C CNN
 F 1 "GND" H 6255 4127 50  0000 C CNN
 F 2 "" H 6250 4300 50  0001 C CNN
@@
 Switched Power Regulator
 $Comp
-L Device:L L?
+L Device:L L501
 U 1 1 5EB90558
 P 6500 3200
-F 0 "L?" V 6600 3350 50  0000 C CNN
+F 0 "L501" V 6600 3350 50  0000 C CNN
 F 1 "1uH" V 6600 3100 50  0000 C CNN
-F 2 "" H 6500 3200 50  0001 C CNN
+F 2 "Inductor_SMD:L_0805_2012Metric_Pad1.15x1.40mm_HandSolder" H 6500 3200 50  0001 C CNN
 F 3 "~" H 6500 3200 50  0001 C CNN
 	1    6500 3200
@@
 	6650 3200 7100 3200
 $Comp
-L rs_Regulator_switching:MIC23155 U?
+L rs_Regulator_switching:MIC23155 U501
 U 1 1 5E6DA7B1
 P 5600 3900
-F 0 "U?" H 5600 4865 50  0000 C CNN
+F 0 "U501" H 5600 4865 50  0000 C CNN
 F 1 "MIC23155" H 5600 4774 50  0000 C CNN
-F 2 "" H 5900 4750 50  0001 C CNN
+F 2 "mic23155:MLF-20-1EP_3x4mm_P0.5mm_EP2.6x1.6mm_thermal_vias" H 5900 4750 50  0001 C CNN
 F 3 "http://ww1.microchip.com/downloads/en/DeviceDoc/MIC23158-59.pdf" H 5900 4750 50  0001 C CNN
 	1    5600 3900
@@
 	5150 3200 5050 3200
 $Comp
-L power:GND #PWR?
+L power:GND #PWR0503
 U 1 1 5E8E7282
 P 4400 3800
-F 0 "#PWR?" H 4400 3550 50  0001 C CNN
+F 0 "#PWR0503" H 4400 3550 50  0001 C CNN
 F 1 "GND" H 4405 3627 50  0000 C CNN
 F 2 "" H 4400 3800 50  0001 C CNN
@@
 $EndComp
 $Comp
-L power:GND #PWR?
+L power:GND #PWR0502
 U 1 1 5E8E700E
 P 4000 3800
-F 0 "#PWR?" H 4000 3550 50  0001 C CNN
+F 0 "#PWR0502" H 4000 3550 50  0001 C CNN
 F 1 "GND" H 4005 3627 50  0000 C CNN
 F 2 "" H 4000 3800 50  0001 C CNN
@@
 	4000 3400 4000 3300
 $Comp
-L power:VBUS #PWR?
+L power:VBUS #PWR0501
 U 1 1 5E8C5758
 P 4000 3300
-F 0 "#PWR?" H 4000 3150 50  0001 C CNN
+F 0 "#PWR0501" H 4000 3150 50  0001 C CNN
 F 1 "VBUS" H 4015 3473 50  0000 C CNN
 F 2 "" H 4000 3300 50  0001 C CNN
@@
 	4000 3400 4400 3400
 $Comp
-L Device:C_Small C?
+L Device:C_Small C501
 U 1 1 5E8C0063
 P 4000 3600
-F 0 "C?" H 4092 3646 50  0000 L CNN
+F 0 "C501" H 4092 3646 50  0000 L CNN
 F 1 "4.7uF" H 4092 3555 50  0000 L CNN
-F 2 "" H 4000 3600 50  0001 C CNN
+F 2 "Capacitor_SMD:C_0603_1608Metric_Pad1.05x0.95mm_HandSolder" H 4000 3600 50  0001 C CNN
 F 3 "~" H 4000 3600 50  0001 C CNN
 	1    4000 3600
@@
 $EndComp
 $Comp
-L Device:C_Small C?
+L Device:C_Small C502
 U 1 1 5E8BFD7C
 P 4400 3600
-F 0 "C?" H 4492 3646 50  0000 L CNN
-F 1 "1uF" H 4492 3555 50  0000 L CNN
-F 2 "" H 4400 3600 50  0001 C CNN
+F 0 "C502" H 4492 3646 50  0000 L CNN
+F 1 "100nF" H 4492 3555 50  0000 L CNN
+F 2 "Capacitor_SMD:C_0603_1608Metric_Pad1.05x0.95mm_HandSolder" H 4400 3600 50  0001 C CNN
 F 3 "~" H 4400 3600 50  0001 C CNN
 	1    4400 3600
@@
 	6050 3600 6600 3600
 Connection ~ 6600 3600
+$Comp
+L Device:C_Small C505
+U 1 1 5E79134A
+P 7500 3600
+F 0 "C505" H 7250 3650 50  0000 L CNN
+F 1 "100nF" H 7150 3550 50  0000 L CNN
+F 2 "Capacitor_SMD:C_0603_1608Metric_Pad1.05x0.95mm_HandSolder" H 7500 3600 50  0001 C CNN
+F 3 "~" H 7500 3600 50  0001 C CNN
+	1    7500 3600
+	1    0    0    -1
+$EndComp
+$Comp
+L power:GND #PWR0102
+U 1 1 5E791AA0
+P 7500 3800
+F 0 "#PWR0102" H 7500 3550 50  0001 C CNN
+F 1 "GND" H 7505 3627 50  0000 C CNN
+F 2 "" H 7500 3800 50  0001 C CNN
+F 3 "" H 7500 3800 50  0001 C CNN
+	1    7500 3800
+	-1   0    0    -1
+$EndComp
+Wire Wire Line
+	7500 3700 7500 3800
+Wire Wire Line
+	7500 3400 7500 3500
+Connection ~ 7500 3400
+Wire Wire Line
+	7500 3400 7700 3400
 $EndSCHEMATC
