File: pcb/module_conector.sch (KiCad schematic (older format))
At the start: 3 parts

Commit message: SCH: minor changes
Parts:
- removed C? (x2): 100nF, symbol Device:C_Small
- removed J?: Conn_02x16_Odd_Even, symbol Connector_Generic:Conn_02x16_Odd_Even
- added J? (x2): Conn_02x06_Odd_Even, symbol Connector_Generic:Conn_02x06_Odd_Even
Connections:
- net +3V3: now also J?.2 (Pin_2), J?.2 (Pin_2)
- net DBUS_0: now also J?.3 (Pin_3)
- net DBUS_1: now also J?.5 (Pin_5)
- net DBUS_2: now also J?.7 (Pin_7)
- net DBUS_3: now also J?.9 (Pin_9)
- net DBUS_4: now also J?.4 (Pin_4)
- net DBUS_5: now also J?.6 (Pin_6)
- net DBUS_6: now also J?.8 (Pin_8)
- net DBUS_7: now also J?.10 (Pin_10)
- net DBUS_MPSSE_0: now also J?.3 (Pin_3)
- net DBUS_MPSSE_1: now also J?.5 (Pin_5)
- net DBUS_MPSSE_2: now also J?.7 (Pin_7)
- net DBUS_MPSSE_3: now also J?.9 (Pin_9)
- net DBUS_MPSSE_4: now also J?.4 (Pin_4)
- net DBUS_MPSSE_5: now also J?.6 (Pin_6)
- net DBUS_MPSSE_6: now also J?.8 (Pin_8)
- net DBUS_MPSSE_7: now also J?.10 (Pin_10)
- net GND: now also J?.11 (Pin_11), J?.11 (Pin_11), J?.12 (Pin_12), J?.12 (Pin_12)
- net VTARGET: now also J?.1 (Pin_1), J?.1 (Pin_1)
- no-connect marks 3 -> 0

Commit message: SCH: slight changes
Parts:
- J701, J702: renamed from J?; footprint (none) -> Connector_PinHeader_2.54mm:PinHeader_2x06_P2.54mm_Vertical
Changed lines of the file:
@@
 	6400 4950 6400 5050
 $Comp
-L power:GND #PWR?
+L power:GND #PWR0704
 U 1 1 5E6A6FBF
 P 6400 5050
-F 0 "#PWR?" H 6400 4800 50  0001 C CNN
+F 0 "#PWR0704" H 6400 4800 50  0001 C CNN
 F 1 "GND" H 6405 4877 50  0000 C CNN
 F 2 "" H 6400 5050 50  0001 C CNN
@@
 	6550 4450 6550 4350
 $Comp
-L power:+3V3 #PWR?
+L power:+3V3 #PWR0706
 U 1 1 5E6B068A
 P 6550 4350
-F 0 "#PWR?" H 6550 4200 50  0001 C CNN
+F 0 "#PWR0706" H 6550 4200 50  0001 C CNN
 F 1 "+3V3" H 6565 4523 50  0000 C CNN
 F 2 "" H 6550 4350 50  0001 C CNN
@@
 	6350 3650 6350 3750
 $Comp
-L power:GND #PWR?
+L power:GND #PWR0703
 U 1 1 5E74F37C
 P 6350 3750
-F 0 "#PWR?" H 6350 3500 50  0001 C CNN
+F 0 "#PWR0703" H 6350 3500 50  0001 C CNN
 F 1 "GND" H 6355 3577 50  0000 C CNN
 F 2 "" H 6350 3750 50  0001 C CNN
@@
 	6500 3150 6500 3050
 $Comp
-L power:+3V3 #PWR?
+L power:+3V3 #PWR0705
 U 1 1 5E74F383
 P 6500 3050
-F 0 "#PWR?" H 6500 2900 50  0001 C CNN
+F 0 "#PWR0705" H 6500 2900 50  0001 C CNN
 F 1 "+3V3" H 6515 3223 50  0000 C CNN
 F 2 "" H 6500 3050 50  0001 C CNN
@@
 	5700 4950 5700 5050
 $Comp
-L power:GND #PWR?
+L power:GND #PWR0702
 U 1 1 5E75B911
 P 5700 5050
-F 0 "#PWR?" H 5700 4800 50  0001 C CNN
+F 0 "#PWR0702" H 5700 4800 50  0001 C CNN
 F 1 "GND" H 5705 4877 50  0000 C CNN
 F 2 "" H 5700 5050 50  0001 C CNN
@@
 $EndComp
 $Comp
-L Connector_Generic:Conn_02x06_Odd_Even J?
+L Connector_Generic:Conn_02x06_Odd_Even J702
 U 1 1 5E75C1C3
 P 6000 4650
-F 0 "J?" H 6050 5067 50  0000 C CNN
+F 0 "J702" H 6050 5067 50  0000 C CNN
 F 1 "Conn_02x06_Odd_Even" H 6050 4976 50  0000 C CNN
-F 2 "" H 6000 4650 50  0001 C CNN
+F 2 "Connector_PinHeader_2.54mm:PinHeader_2x06_P2.54mm_Vertical" H 6000 4650 50  0001 C CNN
 F 3 "~" H 6000 4650 50  0001 C CNN
 	1    6000 4650
@@
 	5650 3650 5650 3750
 $Comp
-L power:GND #PWR?
+L power:GND #PWR0701
 U 1 1 5E76AF74
 P 5650 3750
-F 0 "#PWR?" H 5650 3500 50  0001 C CNN
+F 0 "#PWR0701" H 5650 3500 50  0001 C CNN
 F 1 "GND" H 5655 3577 50  0000 C CNN
 F 2 "" H 5650 3750 50  0001 C CNN
@@
 $EndComp
 $Comp
-L Connector_Generic:Conn_02x06_Odd_Even J?
+L Connector_Generic:Conn_02x06_Odd_Even J701
 U 1 1 5E76C807
 P 5950 3350
-F 0 "J?" H 6000 3767 50  0000 C CNN
+F 0 "J701" H 6000 3767 50  0000 C CNN
 F 1 "Conn_02x06_Odd_Even" H 6000 3676 50  0000 C CNN
-F 2 "" H 5950 3350 50  0001 C CNN
+F 2 "Connector_PinHeader_2.54mm:PinHeader_2x06_P2.54mm_Vertical" H 5950 3350 50  0001 C CNN
 F 3 "~" H 5950 3350 50  0001 C CNN
 	1    5950 3350
